Commit message: adding RPLIDAR Launch, Setting Correct tf dimensions

File: src/car_description/src/description/car_description.urdf (robot description, URDF)
Before this commit: robot fml_car, 5 links, 4 joints
Links:
- removed link front_caster
Joints:
- removed joint caster_joint
- joint base_joint: origin xyz=0.0 0.0 ${-(wheel_radius+wheel_zoff)} rpy=0 0 0 -> xyz=0.0 0.0 ${-(base_height/2)} rpy=0 0 0
- joint imu_joint: origin xyz=0.05 0 0.175 rpy=0 0 0 -> xyz=0.153 0 0.070 rpy=0 0 0; parent base_link -> base_footprint
- joint laser_joint: origin xyz=0.1 0 0.175 rpy=0 0 0 -> xyz=0.165 0 0.152 rpy=0 0 3.14159; parent base_link -> base_footprint
