Commit message: Revisions to Launch files/parameters

File: src/car_slam/src/description/car_description.urdf (robot description, URDF)
Before this commit: robot fml_car, 4 links, 3 joints
Joints:
- joint imu_joint: origin xyz=0.153 0 0.070 rpy=0 0 0 -> xyz=0.153 0 ${0.070-(base_height/2)} rpy=0 0 0; parent base_footprint -> base_link
- joint laser_joint: origin xyz=0.165 0 0.152 rpy=0 0 3.14159 -> xyz=0.165 0 ${0.152-(base_height/2)} rpy=0 0 3.14159; parent base_footprint -> base_link

Commit message: Fix new lidar orientation.

File: src/car_slam/src/description/car_description.urdf (robot description, URDF)
Before this commit: robot fml_car, 4 links, 3 joints
Joints:
- joint laser_joint: origin xyz=0.165 0 ${0.152-(base_height/2)} rpy=0 0 3.14159 -> xyz=0.165 0 ${0.152-(base_height/2)} rpy=0 0 4.712389
